File: DualCANHat.kicad_pcb (KiCad board)
At the start: 2 copper layers, 65 x 56 mm, 5 parts, among them J1 GPIO

Commit message: Made board outline less wide
Other:
- board text removed: "Extend PCB edge 0.5mm if using SMT header"
Changed lines of the file:
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@@
 		)
-	)
-	(gr_arc
-		(start 100 46.5)
-		(mid 100.87868 44.37868)
-		(end 103 43.5)
-		(stroke
-			(width 0.1)
-			(type solid)
-		)
-		(layer "Dwgs.User")
-	)
-	(gr_line
-		(start 100 47)
-		(end 100 46.5)
-		(stroke
-			(width 0.1)
-			(type solid)
-		)
-		(layer "Dwgs.User")
 	)
 	(gr_line
 		(start 100 63)
 		(end 100 81)
-		(stroke
-			(width 0.1)
-			(type solid)
-		)
-		(layer "Dwgs.User")
-	)
-	(gr_line
-		(start 162 43.5)
-		(end 103 43.5)
-		(stroke
-			(width 0.1)
-			(type solid)
-		)
-		(layer "Dwgs.User")
-	)
-	(gr_arc
-		(start 162 43.5)
-		(mid 164.12132 44.37868)
-		(end 165 46.5)
-		(stroke
-			(width 0.1)
-			(type solid)
-		)
-		(layer "Dwgs.User")
-	)
-	(gr_line
-		(start 165 47)
-		(end 165 46.5)
 		(stroke
 			(width 0.1)
@@
 		(layer "Edge.Cuts")
 	)
-	(gr_text "Extend PCB edge 0.5mm if using SMT header"
-		(at 103 42.5 0)
-		(layer "Dwgs.User")
-		(effects
-			(font
-				(size 1 1)
-				(thickness 0.15)
-			)
-			(justify left)
-		)
-	)
 	(gr_text "PoE"

Commit message: Added Libraries folder and changed header to Adafruit 2223
Parts:
- J1: value GPIO -> 2223; footprint Connector_PinSocket_2.54mm:PinSocket_2x20_P2.54mm_Vertical -> Adafruit:RHDR40W64P254X254_2X20_5105X500X865P
- moved J1 2.54 mm to (108.4, 46.2), turned to 0 degrees

Commit message: Placed parts in schematic
Parts:
- added U2: TCAN1044ADDFRQ1, Texas Instruments:DDF0008A-IPC_A, F.Cu at (144.3, 71.5)
- added U3: TCAN1044ADDFRQ1, Texas Instruments:DDF0008A-IPC_A, F.Cu at (126.7, 71.5)
- added U4: MCP2518FDT-E/QBB, Microchip:VDFN14_QBB_MCH, F.Cu at (127.0, 60.0)
- added U5: MCP2518FDT-E/QBB, Microchip:VDFN14_QBB_MCH, F.Cu at (144.6, 60.3)
Other:
- outline, holes or cut-outs redrawn
- board text removed: "DISPLAY (OPTIONAL)"
